File: Master2.kicad_pcb (KiCad board)
At the start: 2 copper layers, 49 parts, among them J1 Conn_01x16_Socket, J10 Conn_01x08_Socket, J11 Conn_01x08_Socket, J12 Conn_01x07_Pin, J13 Screw_Terminal_01x06, J14 Screw_Terminal_01x06, J15 Screw_Terminal_01x06, J16 Screw_Terminal_01x06, J2 XT60-M, J3 Conn_01x06_Socket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

Commit message: PCB
Parts:
- removed D1: 1N62xxA, Diode_THT:D_DO-201AE_P15.24mm_Horizontal
- SW2: footprint Button_Switch_THT:SW_DIP_SPSTx01_Slide_6.7x4.1mm_W7.62mm_P2.54mm_LowProfile -> Button_Switch_THT:SW_E-Switch_EG1224_SPDT_Angled
- moved SW2 9.44 mm to (145.7, 152.1), turned to 90 degrees
Connections:
- SW2 pad 1: Net-(J2-POS) -> vcc
- SW2 pad 2: Net-(D1-A2) -> Net-(J2-POS)
Routing:
- net Net-(D1-A2): track 8.93 -> 0.00 mm
- net Net-(J2-POS): track 9.40 -> 18.1 mm
- net vcc: track 12.5 -> 9.63 mm
