File: Master2.kicad_sch (KiCad schematic)
At the start: 49 parts, among them J1 Conn_01x16_Socket, J10 Conn_01x08_Socket, J11 Conn_01x08_Socket, J12 Conn_01x07_Pin, J13 Screw_Terminal_01x06, J14 Screw_Terminal_01x06, J15 Screw_Terminal_01x06, J16 Screw_Terminal_01x06, J2 XT60-M, J3 Conn_01x06_Socket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

Commit message: PCB
Parts:
- removed D1: 1N62xxA, Diode_THT:D_DO-201AE_P15.24mm_Horizontal, symbol Diode:1N62xxA
- SW2: footprint Button_Switch_THT:SW_DIP_SPSTx01_Slide_6.7x4.1mm_W7.62mm_P2.54mm_LowProfile -> Button_Switch_THT:SW_E-Switch_EG1224_SPDT_Angled; symbol Switch:SW_SPST -> Switch:SW_SPDT_MSM
Connections:
- net vcc: now also SW2.1
- net at SW2.2: now also J2.P (POS)
Changed lines of the file:
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@@
     )
   )
-  (global_label "vcc" (shape input) (at 187.96 82.55 0) (fields_autoplaced)
-    (effects (font (size 1.27 1.27)) (justify left))
-    (property "Intersheetrefs" "${INTERSHEET_REFS}" (at 194.0106 82.55 0)
+  (global_label "vcc" (shape input) (at 180.34 80.01 0) (fields_autoplaced)
+    (effects (font (size 1.27 1.27)) (justify left))
+    (property "Intersheetrefs" "${INTERSHEET_REFS}" (at 186.3906 80.01 0)
       (effects (font (size 1.27 1.27)) (justify left) hide)
     )
@@
     )
   )
-  (symbol (lib_id "Diode:1N62xxA") (at 184.15 82.55 180) (unit 1)
-    (in_bom yes) (on_board yes) (dnp no) (fields_autoplaced)
-    (property "Reference" "D1" (at 184.15 77.47 0)
-      (effects (font (size 1.27 1.27)))
-    )
-    (property "Value" "1N62xxA" (at 184.15 80.01 0)
-      (effects (font (size 1.27 1.27)))
-    )
-    (property "Footprint" "Diode_THT:D_DO-201AE_P15.24mm_Horizontal" (at 184.15 77.47 0)
-      (effects (font (size 1.27 1.27)) hide)
-    )
-    (property "Datasheet" "https://www.vishay.com/docs/88301/15ke.pdf" (at 185.42 82.55 0)
-      (effects (font (size 1.27 1.27)) hide)
-    )
-    (pin "1")
-    (pin "2")
-    (instances
-      (project "Master2"
-        (path "/2ccf91c7-fc26-4b60-b5c9-bd6619eae593"
-          (reference "D1") (unit 1)
-        )
-      )
-    )
-  )
   (symbol (lib_id "Transistor_BJT:TIP2955") (at 173.99 104.14 270) (mirror x) (unit 1)
     (in_bom yes) (on_board yes) (dnp no)
@@
     )
   )
-  (symbol (lib_id "Switch:SW_SPST") (at 175.26 82.55 0) (unit 1)
+  (symbol (lib_id "Switch:SW_SPDT_MSM") (at 175.26 82.55 0) (unit 1)
     (in_bom yes) (on_board yes) (dnp no) (fields_autoplaced)
     (property "Reference" "SW2" (at 175.26 77.47 0)
@@
     )
     (property "Value" "SW_SPST" (at 175.26 80.01 0)
-      (effects (font (size 1.27 1.27)))
-    )
-    (property "Footprint" "Button_Switch_THT:SW_DIP_SPSTx01_Slide_6.7x4.1mm_W7.62mm_P2.54mm_LowProfile" (at 175.26 82.55 0)
+      (effects (font (size 1.27 1.27)) hide)
+    )
+    (property "Footprint" "Button_Switch_THT:SW_E-Switch_EG1224_SPDT_Angled" (at 175.26 82.55 0)
       (effects (font (size 1.27 1.27)) hide)
     )
@@
     (pin "1")
     (pin "2")
-    (instances
-      (project "Master2"
+    (pin "3")
+    (instances
+      (project "Master2"
